File: 01_DESIGN/kicad_demo_project/AVR.kicad_sch (KiCad schematic)
At the start: 20 parts, among them J4 JP2, J5 JP8, U5 OPA2340UA, U6 ATMEGA324PA, Y2 8MHz

Commit message: Update schematic, PCB
Parts:
- removed C33: 0.1uF/6.3V, CAP_C_1608X80, symbol Altium_Lib_by_KhueNguyenCreator:root_1_Tu 0402 33nF 10V_Altium_Lib_by_KhueNguye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
- removed J4: JP2, Connector_PinHeader_2.54mm:PinHeader_1x02_P2.54mm_Horizontal, symbol TechMT.VN_Lib:root_0_mirrored_JP2_TechMT.VN_Lib.IntLib
- removed J5: JP8, Connector_PinHeader_2.54mm:PinHeader_1x08_P2.54mm_Horizontal, symbol obc_ver2:root_0_JP8_obc_ver2.SCHLIB
- removed U5: OPA2340UA, SOIC127P602X173-8N, symbol Sang_library:root_0_OPA2340UA/2K5_Sang_library.SchLib
- removed Y2: 8MHz, Crystal:Crystal_SMD_3225-4Pin_3.2x2.5mm, symbol ECS-250-12-33Q-JES-TR:root_0_ECS-250-12-33Q-JES-TR_ECS-250-12-33Q-JES-TR.IntLib
- added C58: 0.1uF/6.3V, Capacitor_SMD:C_0603_1608Metric, symbol Device:C
- added J5: Conn_01x08, Connector_PinHeader_2.54mm:PinHeader_1x08_P2.54mm_Vertical, symbol Connector_Generic:Conn_01x08
- added J6: Conn_01x02, Connector_PinHeader_2.54mm:PinHeader_1x02_P2.54mm_Vertical, symbol Connector_Generic:Conn_01x02
- added U5: OPA2340, Package_SO:SOIC-8_3.9x4.9mm_P1.27mm, symbol Amplifier_Operational:OPA2340
- added Y2: Crystal_GND24, Crystal:Crystal_SMD_3225-4Pin_3.2x2.5mm, symbol Device:Crystal_GND24
- C34, C35, C38, C39, C40, C41, C42: footprint CAP_C_1608X80 -> Capacitor_SMD:C_0603_1608Metric; symbol Altium_Lib_by_KhueNguyenCreator:root_1_Tu 0402 33nF 10V_Altium_Lib_by_KhueNguyenCreator.IntLib -> Device:C
- C36, C37: footprint CAP_C_1608X80 -> Capacitor_SMD:C_0603_1608Metric; symbol Altium_Lib_by_KhueNguyenCreator:root_3_mirrored_Tu 0402 33nF 10V_Altium_Lib_by_KhueNguyenCreator.IntLib -> Device:C
- L1: footprint RES_C_1608X60 -> Inductor_SMD:L_0603_1608Metric; symbol Sang_library:root_0_L-SMD-1_Sang_library.SchLib -> Device:L
- R15, R16: footprint RES_C_1608X60 -> Resistor_SMD:R_0603_1608Metric; symbol Altium_Lib_by_KhueNguyenCreator:root_2_Tro 0603 1% 10k_Altium_Lib_by_KhueNguyenCreator.IntLib -> Device:R
- R17: footprint RES_C_1608X60 -> Resistor_SMD:R_0603_1608Metric; symbol Altium_Lib_by_KhueNguyenCreator:root_3_Tro 0603 1% 10k_Altium_Lib_by_KhueNguyenCreator.IntLib -> Device:R
- R18: footprint RES_C_1608X60 -> Resistor_SMD:R_0603_1608Metric; symbol Altium_Lib_by_KhueNguyenCreator:root_1_Tro 0603 1% 10k_Altium_Lib_by_KhueNguyenCreator.IntLib -> Device:R
- U6: symbol AUSB:root_0_MCU_ATMEGA324PA_AUSB.SchLib -> ausb:ATMEGA324PA; Manufacturer (none) -> Microchip Technology; Manufacturer Part Number (none) -> ATMEGA324PA-AU; Supplier (none) -> Digikey; Supplier Part Number (none) -> ATMEGA324PA-AU-ND
Connections:
- net +5V: now also C38.2, C39.2, C40.2, C42.2, C58.1, J5.1 (Pin_1), J6.1 (Pin_1), U5.8 (V+); no longer C38.1, C39.1, C40.1, C42.1
- net +5V_AVCC: now also C41.2; no longer C41.1
- net ADC_TEMP1: now also C34.2; no longer C34.1
- net AVR_JTAG_TCK: now also J5.5 (Pin_5)
- net AVR_JTAG_TDI: now also J5.3 (Pin_3)
- net AVR_JTAG_TDO: now also J5.6 (Pin_6)
- net AVR_JTAG_TMS: now also J5.4 (Pin_4)
- net AVR_JTAG_nRESET: now also J5.8 (Pin_8)
- net GND: now also C34.1, C35.1, C36.2, C37.2, C38.1, C39.1, C40.1, C41.1, C42.1, C58.2, J5.2 (Pin_2), J5.7 (Pin_7), U5.4 (V-), Y2.2 (G), Y2.4 (G); no longer C34.2, C35.2, C36.1, C37.1, C38.2, C39.2, C40.2, C41.2, C42.2
- net NTC1-: now also J6.2 (Pin_2)
- net at R15.2: now also U5.1, U5.2 (-)
- net at U6.7 (XTAL2): now also C36.1, Y2.1; no longer C36.2
- net at U6.8 (XTAL1): now also C37.1, Y2.3; no longer C37.2
- net at R16.1: now also C35.2, U5.3 (+); no longer C35.1
- no-connect marks 19 -> 21
Other:
- moved on the sheet: R15, R18, U6
