File: 01_DESIGN/kicad_demo_project/eMMC.kicad_sch (KiCad schematic)
At the start: 20 parts, among them U4 MTFC32GAZAQDW-AAT

Commit message: Update schematic, PCB
Parts:
- removed C52, C53: 4.7uF/6.3V, CAP_MP_1608X90, symbol TACL335M003RTA:root_1_mirrored_TACL335M003RTA_TACL335M003RTA.IntLib
- added C52, C53: 4.7uF, Capacitor_Tantalum_SMD:CP_EIA-1608-10_AVX-L, symbol Device:C_Polarized_US
- C27, C30, C32, C46, C47, C48, C49, C50, C51: footprint CAP_C_1608X80 -> Capacitor_SMD:C_0603_1608Metric; symbol Altium_Lib_by_KhueNguyenCreator:root_1_Tu 0402 33nF 10V_Altium_Lib_by_KhueNguyenCreator.IntLib -> Device:C
- C31: footprint CAP_MP_1608X90 -> Capacitor_SMD:C_0603_1608Metric; symbol TACL335M003RTA:root_1_mirrored_TACL335M003RTA_TACL335M003RTA.IntLib -> Device:C
- R10, R11, R12, R13, R8, R9: footprint RES_C_1608X60 -> Resistor_SMD:R_0603_1608Metric; symbol Altium_Lib_by_KhueNguyenCreator:root_1_Tro 0603 1% 10k_Altium_Lib_by_KhueNguyenCreator.IntLib -> Device:R
- R14: footprint RES_C_1608X60 -> Resistor_SMD:R_0603_1608Metric; symbol Altium_Lib_by_KhueNguyenCreator:root_0_Tro 0603 1% 10k_Altium_Lib_by_KhueNguyenCreator.IntLib -> Device:R
- U4: footprint BGA_100_C_100P_10X17_1400X1800X150 -> Package_BGA:BGA-100_14x18mm_Layout10x17_P1mm; symbol emmc_nofootprint:root_0_MTFC32GAZAQDW-AAT_emmc_nofootprint.IntLib -> ausb:MTFC32GAZAQDW-AAT
Connections:
- net +3.3V: now also C27.2, C32.2, C46.2, C47.2, C48.2, C49.2, C50.2, C51.2, C52.1, C53.1; no longer C27.1, C32.1, C46.1, C47.1, C48.1, C49.1, C50.1, C51.1
- net GND: now also C27.1, C30.1, C31.1, C32.1, C46.1, C47.1, C48.1, C49.1, C50.1, C51.1, C52.2, C53.2; no longer C27.2, C30.2, C31.2, C32.2, C46.2, C47.2, C48.2, C49.2, C50.2, C51.2
- new net: C30.2, C31.2, U4.E4 (VDDIM)
Other:
- moved on the sheet: R10, R11, R12, R13, R14, R8, R9, U4A, U4B, U4C
